File: Education/2019/pcbIsolationMilling/eagle/eagle2_hotovo.brd (EAGLE design)
At the start: 100 x 80 mm, 11 parts, among them IC1 555

Commit message: finalized workshop
Other:
- board size 100 x 80 mm -> 45.4 x 29.2 mm
Changed lines of the file:
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@@
 <board>
 <plain>
-<wire x1="0" y1="0" x2="100" y2="0" width="0" layer="20"/>
-<wire x1="100" y1="0" x2="100" y2="80" width="0" layer="20"/>
-<wire x1="100" y1="80" x2="0" y2="80" width="0" layer="20"/>
-<wire x1="0" y1="80" x2="0" y2="0" width="0" layer="20"/>
+<wire x1="10.16" y1="40.64" x2="55.55" y2="40.64" width="0" layer="20"/>
+<wire x1="55.55" y1="40.64" x2="55.55" y2="69.84" width="0" layer="20"/>
+<wire x1="55.55" y1="69.84" x2="10.16" y2="69.84" width="0" layer="20"/>
+<wire x1="10.16" y1="69.84" x2="10.16" y2="40.64" width="0" layer="20"/>
 </plain>
 <attributes>
